File: Hardware/UDAWA-Aktuator4CH/UDAWA-Aktuator4CH.sch (EAGLE design)
At the start: 3 parts

Commit message: #3 to do list 6&7
Parts:
- added CH1, CH2, CH3, CH4, NO1, NO3: (no value), con-wago-500:W237-102
Connections:
- new net NO1: CH1-1.KL, NO1-1.KL
- new net NO2: CH2-1.KL, NO1-2.KL
- new net NO3: CH3-1.KL, NO3-1.KL
- new net NO4: CH4-1.KL, NO3-2.KL
Changed lines of the file:
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@@
 <part name="HLK1" library="HLK-PM01" deviceset="HLK-PM01" device="3W"/>
 <part name="220V" library="con-wago-500" library_urn="urn:adsk.eagle:library:195" deviceset="W237-102" device="" package3d_urn="urn:adsk.eagle:package:10688/1"/>
+<part name="NO1" library="con-wago-500" library_urn="urn:adsk.eagle:library:195" deviceset="W237-102" device="" package3d_urn="urn:adsk.eagle:package:10688/1"/>
+<part name="NO3" library="con-wago-500" library_urn="urn:adsk.eagle:library:195" deviceset="W237-102" device="" package3d_urn="urn:adsk.eagle:package:10688/1"/>
+<part name="CH1" library="con-wago-500" library_urn="urn:adsk.eagle:library:195" deviceset="W237-102" device="" package3d_urn="urn:adsk.eagle:package:10688/1"/>
+<part name="CH3" library="con-wago-500" library_urn="urn:adsk.eagle:library:195" deviceset="W237-102" device="" package3d_urn="urn:adsk.eagle:package:10688/1"/>
+<part name="CH2" library="con-wago-500" library_urn="urn:adsk.eagle:library:195" deviceset="W237-102" device="" package3d_urn="urn:adsk.eagle:package:10688/1"/>
+<part name="CH4" library="con-wago-500" library_urn="urn:adsk.eagle:library:195" deviceset="W237-102" device="" package3d_urn="urn:adsk.eagle:package:10688/1"/>
 </parts>
 <sheets>
@@
 <attribute name="VALUE" x="-45.72" y="16.637" size="1.778" layer="96"/>
 <attribute name="NAME" x="-43.18" y="21.209" size="1.778" layer="95" rot="R180"/>
+</instance>
+<instance part="NO1" gate="-1" x="-60.96" y="-15.24" smashed="yes">
+<attribute name="NAME" x="-60.96" y="-14.351" size="1.778" layer="95" rot="R180"/>
+</instance>
+<instance part="NO1" gate="-2" x="-60.96" y="-20.32" smashed="yes">
+<attribute name="VALUE" x="-63.5" y="-24.003" size="1.778" layer="96"/>
+<attribute name="NAME" x="-60.96" y="-19.431" size="1.778" layer="95" rot="R180"/>
+</instance>
+<instance part="NO3" gate="-1" x="-60.96" y="-25.4" smashed="yes">
+<attribute name="NAME" x="-60.96" y="-24.511" size="1.778" layer="95" rot="R180"/>
+</instance>
+<instance part="NO3" gate="-2" x="-60.96" y="-30.48" smashed="yes">
+<attribute name="VALUE" x="-63.5" y="-34.163" size="1.778" layer="96"/>
+<attribute name="NAME" x="-60.96" y="-29.591" size="1.778" layer="95" rot="R180"/>
+</instance>
+<instance part="CH1" gate="-1" x="-25.4" y="-22.86" smashed="yes">
+<attribute name="NAME" x="-25.4" y="-21.971" size="1.778" layer="95" rot="R180"/>
+</instance>
+<instance part="CH1" gate="-2" x="-25.4" y="-27.94" smashed="yes">
+<attribute name="VALUE" x="-27.94" y="-31.623" size="1.778" layer="96"/>
+<attribute name="NAME" x="-25.4" y="-27.051" size="1.778" layer="95" rot="R180"/>
+</instance>
+<instance part="CH3" gate="-1" x="-25.4" y="-43.18" smashed="yes">
+<attribute name="NAME" x="-25.4" y="-42.291" size="1.778" layer="95" rot="R180"/>
+</instance>
+<instance part="CH3" gate="-2" x="-25.4" y="-48.26" smashed="yes">
+<attribute name="VALUE" x="-27.94" y="-51.943" size="1.778" layer="96"/>
+<attribute name="NAME" x="-25.4" y="-47.371" size="1.778" layer="95" rot="R180"/>
+</instance>
+<instance part="CH2" gate="-1" x="-25.4" y="-33.02" smashed="yes">
+<attribute name="NAME" x="-25.4" y="-32.131" size="1.778" layer="95" rot="R180"/>
+</instance>
+<instance part="CH2" gate="-2" x="-25.4" y="-38.1" smashed="yes">
+<attribute name="VALUE" x="-27.94" y="-41.783" size="1.778" layer="96"/>
+<attribute name="NAME" x="-25.4" y="-37.211" size="1.778" layer="95" rot="R180"/>
+</instance>
+<instance part="CH4" gate="-1" x="-25.4" y="-53.34" smashed="yes">
+<attribute name="NAME" x="-25.4" y="-52.451" size="1.778" layer="95" rot="R180"/>
+</instance>
+<instance part="CH4" gate="-2" x="-25.4" y="-58.42" smashed="yes">
+<attribute name="VALUE" x="-27.94" y="-62.103" size="1.778" layer="96"/>
+<attribute name="NAME" x="-25.4" y="-57.531" size="1.778" layer="95" rot="R180"/>
 </instance>
 </instances>
@@
 </segment>
 </net>
+<net name="NO2" class="0">
+<segment>
+<pinref part="NO1" gate="-2" pin="KL"/>
+<wire x1="-55.88" y1="-20.32" x2="-53.34" y2="-20.32" width="0.1524" layer="91"/>
+<label x="-53.34" y="-20.32" size="1.778" layer="95" xref="yes"/>
+</segment>
+<segment>
+<pinref part="CH2" gate="-1" pin="KL"/>
+<wire x1="-20.32" y1="-33.02" x2="-17.78" y2="-33.02" width="0.1524" layer="91"/>
+<label x="-17.78" y="-33.02" size="1.778" layer="95" xref="yes"/>
+</segment>
+</net>
+<net name="NO4" class="0">
+<segment>
+<pinref part="NO3" gate="-2" pin="KL"/>
+<wire x1="-55.88" y1="-30.48" x2="-53.34" y2="-30.48" width="0.1524" layer="91"/>
+<label x="-53.34" y="-30.48" size="1.778" layer="95" xref="yes"/>
+</segment>
+<segment>
+<pinref part="CH4" gate="-1" pin="KL"/>
+<wire x1="-20.32" y1="-53.34" x2="-17.78" y2="-53.34" width="0.1524" layer="91"/>
+<label x="-17.78" y="-53.34" size="1.778" layer="95" xref="yes"/>
+</segment>
+</net>
+<net name="NO3" class="0">
+<segment>
+<pinref part="CH3" gate="-1" pin="KL"/>
+<wire x1="-20.32" y1="-43.18" x2="-17.78" y2="-43.18" width="0.1524" layer="91"/>
+<label x="-17.78" y="-43.18" size="1.778" layer="95" xref="yes"/>
+</segment>
+<segment>
+<pinref part="NO3" gate="-1" pin="KL"/>
+<wire x1="-55.88" y1="-25.4" x2="-53.34" y2="-25.4" width="0.1524" layer="91"/>
+<label x="-53.34" y="-25.4" size="1.778" layer="95" xref="yes"/>
+</segment>
+</net>
+<net name="NO1" class="0">
+<segment>
+<pinref part="NO1" gate="-1" pin="KL"/>
+<wire x1="-55.88" y1="-15.24" x2="-53.34" y2="-15.24" width="0.1524" layer="91"/>
+<label x="-53.34" y="-15.24" size="1.778" layer="95" xref="yes"/>
+</segment>
+<segment>
+<pinref part="CH1" gate="-1" pin="KL"/>
+<wire x1="-20.32" y1="-22.86" x2="-17.78" y2="-22.86" width="0.1524" layer="91"/>
+<label x="-17.78" y="-22.86" size="1.778" layer="95" xref="yes"/>
+</segment>
+</net>
